File: kicadFiles/austin.kicad_pcb (KiCad board)
At the start: 2 copper layers, 391.5 x 134 mm, 465 parts, among them J1 TYPE-C-31-M12_13, J2 Conn_01x04_Male, J5 Conn_01x06_Male, Q1 AO4406AL, SW1 MXSwitch, SW10 MXSwitch, SW100 MXSwitch, SW101 MXSwitch, SW102 MXSwitch, SW103 MXSwitch, SW104 MXSwitch, SW105 MXSwitch, SW106 MXSwitch, SW107 MXSwitch, SW108 MXSwitch, SW109 MXSwitch, SW11 MXSwitch, SW110 MXSwitch, SW111 MXSwitch, SW112 MXSwitch, SW12 MXSwitch, SW13 MXSwitch, SW14 MXSwitch, SW15 MXSwitch, SW16 MXSwitch, SW17 MXSwitch, SW18 MXSwitch, SW19 MXSwitch, SW2 MXSwitch, SW20 MXSwitch, SW21 MXSwitch, SW22 MXSwitch, SW23 MXSwitch, SW24 MXSwitch, SW25 MXSwitch, SW26 MXSwitch, SW27 MXSwitch, SW28 MXSwitch, SW29 MXSwitch, SW3 MXSwitch, SW30 MXSwitch, SW31 MXSwitch, SW32 MXSwitch, SW33 MXSwitch, SW34 MXSwitch, SW35 MXSwitch, SW36 MXSwitch, SW37 MXSwitch, SW38 MXSwitch, SW39 MXSwitch, SW4 MXSwitch, SW40 MXSwitch, SW41 MXSwitch, SW42 MXSwitch, SW43 MXSwitch, SW44 MXSwitch, SW45 MXSwitch, SW46 MXSwitch, SW47 MXSwitch, SW48 MXSwitch, SW49 MXSwitch, SW5 MXSwitch, SW50 MXSwitch, SW51 MXSwitch, SW52 MXSwitch, SW53 MXSwitch, SW54 MXSwitch, SW55 MXSwitch, SW56 MXSwitch, SW57 MXSwitch, SW58 MXSwitch, SW59 MXSwitch, SW6 MXSwitch, SW60 MXSwitch, SW61 MXSwitch, SW62 MXSwitch, SW63 MXSwitch, SW64 MXSwitch, SW65 MXSwitch, SW66 MXSwitch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

Commit message: [Pre-release] V1.0 pre-release
Parts:
- removed CSin1, CSout1, CVB2, CVB3: 100n, Capacitor_SMD:C_0805_2012Metric_Pad1.15x1.40mm_HandSolder
- removed CVB4: 1u, Capacitor_SMD:C_0805_2012Metric_Pad1.15x1.40mm_HandSolder
- removed CVB5: 4.7u, Capacitor_SMD:C_0805_2012Metric_Pad1.15x1.40mm_HandSolder
- added CB2: 100n, Capacitor_SMD:C_0805_2012Metric_Pad1.15x1.40mm_HandSolder, F.Cu at (175.1, 74.5)
- added CB3: 100n, Capacitor_SMD:C_0805_2012Metric_Pad1.15x1.40mm_HandSolder, F.Cu at (159.7, 73.2)
- added CB4: 100n, Capacitor_SMD:C_0805_2012Metric_Pad1.15x1.40mm_HandSolder, F.Cu at (156.7, 79.9)
- added CB5: 10u, Capacitor_SMD:C_0805_2012Metric_Pad1.15x1.40mm_HandSolder, F.Cu at (158.9, 79.9)
- added CRI1: 100n, Capacitor_SMD:C_0805_2012Metric_Pad1.15x1.40mm_HandSolder, B.Cu at (192.6, 80.0)
- added CRO1: 100n, Capacitor_SMD:C_0805_2012Metric_Pad1.15x1.40mm_HandSolder, B.Cu at (185.6, 80.0)
- added LEDCAPS1: LED, acheronComponents:thtLED, F.Cu at (153.3, 149.5)
- added LEDNUM1: LED, acheronComponents:thtLED, F.Cu at (151.2, 153.2)
- added LEDSCRL1: LED, acheronComponents:thtLED, F.Cu at (155.5, 153.2)
- added RI1: 360, acheronComponents:R_1026, B.Cu at (158.1, 149.5)
- added RI2: 360, acheronComponents:R_1026, B.Cu at (163.1, 149.5)
- added RI3: 360, acheronComponents:R_1026, B.Cu at (160.6, 149.5)
- CB1: renamed from CVB1; moved to F.Cu
- Q1: moved to F.Cu
- RGP: renamed from RPGate1; moved to F.Cu
- RGS: renamed from RSGate1; moved to F.Cu
- RL107, RL94: moved to B.Cu
- SW111: footprint acheronKeyboardSwitches:MX700 -> acheronKeyboardSwitches:MX700R
- moved CRST2 24.4 mm to (135.8, 79.6)
- moved SWRST 24.4 mm to (127.5, 79.6)
- moved CRST1 24.4 mm to (151.7, 79.7)
- moved DRST 24.4 mm to (148.0, 79.7)
- moved QRST 24.4 mm to (140.6, 79.6)
- moved RRST 24.4 mm to (145.6, 79.7)
- moved RGS 23.2 mm to (169.2, 146.8), turned to 270 degrees
- moved D16 21.6 mm to (122.2, 62.0), turned to 270 degrees
- moved U2 21.3 mm to (189.1, 80.0), turned to 180 degrees
- moved RGP 20.8 mm to (166.8, 146.8), turned to 90 degrees
- moved Q1 16.3 mm to (160.9, 146.8), turned to 180 degrees
- moved DS33 16.2 mm to (181.1, 80.0), turned to 270 degrees
- moved DF1 15.4 mm to (275.6, 64.7)
- moved F1 15.4 mm to (269.6, 64.7)
- moved RL107 15.2 mm to (75.1, 174.5), turned to 0 degrees
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- renumbered CUSB1 to CUSB, D63 to D100, D65 to D101, D66 to D102, D71 to D103, D79 to D104, D85 to D105, D91 to D106, D97 to D107, D103 to D108, D67 to D13, D72 to D14, D75 to D15, D80 to D16, D86 to D17, D92 to D18, D98 to D19, D13 to D20, D14 to D21, D15 to D22, D16 to D23, D17 to D24, D18 to D25, D19 to D26, D20 to D27, D21 to D28, D22 to D29, D23 to D30, D24 to D31, D68 to D32, D73 to D33, D76 to D35, D81 to D36, D87 to D37, D93 to D38, D99 to D39, D25 to D40, D26 to D41, D27 to D42, D28 to D43, D29 to D44, D30 to D45, D31 to D46, D32 to D47, D33 to D48, D34 to D49, D35 to D50, D36 to D51, D69 to D52, D74 to D53, D77 to D54, D82 to D55, D88 to D56, D94 to D57, D100 to D59, D37 to D61, D38 to D62, D39 to D63, D40 to D64, D41 to D65, D42 to D66, D43 to D67, D44 to D68, D45 to D69, D46 to D70, D47 to D71, D104 to D72, D48 to D73, D78 to D74, D83 to D75, D89 to D76, D95 to D77, D101 to D78, D49 to D79, D51 to D80, D53 to D81, D55 to D82, D56 to D83, D57 to D84, D59 to D85, D60 to D86, D61 to D87, D62 to D88, D64 to D89, D105 to D90, D70 to D91, D84 to D92, D90 to D93, D96 to D94, D102 to D95, D50 to D96, D52 to D97, D54 to D98, D58 to D99, DRST1 to DRST, QRST1 to QRST, RCC1 to RCC, R72 to RL72, RRST1 to RRST, SWRST1 to SWRST
Connections:
- U1 pad 10: Col6 -> Net-(U1-Pad10)
- U1 pad 11: Row6 -> Row2
- U1 pad 12: Row2 -> Col16
- U1 pad 13: Col5 -> CAPSLCK
- U1 pad 14: Row5 -> NUMLCK
- U1 pad 15: Row4 -> Col10
- U1 pad 17: Col1 -> Row4
- U1 pad 18: Col10 -> Row5
- U1 pad 19: Col11 -> Row6
- U1 pad 20: Col12 -> Col1
- U1 pad 21: Col13 -> Col2
- U1 pad 26: Col9 -> Col4
- U1 pad 27: Col8 -> Col5
- U1 pad 28: Col7 -> Col6
- U1 pad 29: Net-(U1-Pad29) -> Col7
- U1 pad 3: Net-(U1-Pad3) -> Col18
- U1 pad 30: Col4 -> Col8
- U1 pad 31: Col2 -> Col9
- U1 pad 38: Col14 -> Col11
- U1 pad 39: Col19 -> Col12
- U1 pad 4: Net-(U1-Pad4) -> Col17
- U1 pad 40: Col18 -> Col13
- U1 pad 41: Col17 -> Col14
- U1 pad 45: Col16 -> Col15
- U1 pad 46: Col15 -> Net-(U1-Pad46)
- U1 pad 5: Net-(U1-Pad5) -> SCRLLCK
- U1 pad 6: Net-(U1-Pad6) -> Col19
Routing:
- net Row6: track 668.1 -> 1010.2 mm, vias 3 -> 0
- net Row4: track 411.6 -> 735.3 mm, vias 2 -> 0
- net Row3: track 412.6 -> 722.5 mm, vias 2 -> 0
- net Row5: track 465.5 -> 774.6 mm, vias 2 -> 0
- net Col1: track 202.1 -> 489.2 mm
- net Col2: track 206.5 -> 451.0 mm
- net Col3: track 168.2 -> 410.9 mm
- net Col4: track 148.1 -> 376.9 mm
- net Col5: track 148.1 -> 351.3 mm
- net Col6: track 222.2 -> 407.0 mm
- net /LEDK: track 2701.6 -> 2880.2 mm
- net Col7: track 148.1 -> 315.8 mm
- net Col8: track 148.1 -> 288.8 mm
- net Col9: track 141.9 -> 264.9 mm
- net SWDIO: track 0.00 -> 107.5 mm, vias 0 -> 1
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Other:
- board size 391.5 x 134 mm -> 391.5 x 131 mm
- net class Fine removed
- board text added: "1U BKSP"
- board text added: "1U ZERO"
- board text added: "2U BKSP"
- board text added: "2U ZERO"
- board text added: "AustinPCB V1.0 Designed by Gondolindrim In partnership with driftingbunnies and PheonixStar "yea mate lit""
- board text added: "CAPS LOCK"
- board text added: "NUM LOCK"
- board text added: "SCROLL LOCK"
- board text added: "TRACE WIDTH: 0.25mm (approx. 10mil)"
- board text added: "TRACE WIDTH: 0.5mm"
- board text added: "VIA HOLE SIZE (DRILL): 0.3mm"
- board text added: "VIA-TO-VIA AND VIA-TO-TRACE CLEARANCE: 0.25mm (approx. 10mil)"
- board text removed: "AustinPCB V0.1 Designed by Gondolindrim In partnership with driftingbunnies and PhoenixStar "yea mate lit""
- board text removed: "TRACE WIDTH: 0.13mm (approx. 5mil)"
- board text removed: "TRACE WIDTH: 0.25mm"
- board text removed: "VIA HOLE SIZE (DRILL): 0.2mm"
- board text removed: "VIA-TO-VIA AND VIA-TO-TRACE CLEARANCE: 0.13mm (approx. 5mil)"

Commit message: [Update] Version 1.1
Parts:
- U2: value MCP1700-3302E_SOT23 -> TLV1117-33; footprint Package_TO_SOT_SMD:SOT-23 -> Package_TO_SOT_SMD:SOT-223-3_TabPin2
- U3: footprint Package_TO_SOT_SMD:SOT-23-6 -> acheronComponents:SOT-23-6
- moved CRI1 6.75 mm to (199.3, 80.0)
- moved L2 6.00 mm to (254.1, 80.0)
- moved U2 2.00 mm to (191.1, 80.0)
- moved CRO1 1.50 mm to (184.1, 80.0)
- moved RGS 0.10 mm to (169.3, 146.8)
- moved U3 0.07 mm to (274.6, 71.5)
- renumbered SWRST to SWRST1
Routing:
- net 3.3V: track 163.2 -> 168.6 mm
- net GND: track 43.0 -> 46.0 mm
- net Col18: track 292.9 -> 292.1 mm
- net Net-(D105-Pad2): track 15.1 -> 14.4 mm
- net Col12: track 208.8 -> 208.1 mm
- net Net-(D16-Pad2): track 18.4 -> 17.9 mm
Other:
- board text added: "1U PLUS"
- board text added: "2U PLUS"
- board text added: "AustinPCB V1.1 Designed by Gondolindrim In partnership with driftingbunnies and PheonixStar "yea mate lit""
- board text removed: "AustinPCB V1.0 Designed by Gondolindrim In partnership with driftingbunnies and PheonixStar "yea mate lit""

Commit message: [Update] V1.2: plated logo, new easter egg
Parts:
- added L1: Logo, austinLogo:austinLogo_16x40_Plated, F.Cu at (288.6, 168.5)
Routing:
- net Net-(D99-Pad2): track 14.1 -> 12.5 mm
Other:
- board text added: "AustinPCB V1.2 Designed by Gondolindrim In partnership with driftingbunnies and PheonixStar "this burger tastes like sorbothane""
- board text removed: "AustinPCB V1.1 Designed by Gondolindrim In partnership with driftingbunnies and PheonixStar "yea mate lit""
